Commit message: release: publish current NezhaSim workspace
Upload the maintained ROS 1/Gazebo simulator tree, repair clone and submodule metadata, correct the hands-on tutorials, and add the NezhaSim2 preview.

File: src/nezha_sim/nezha_description/nezha_beetle/UAV/nezha_beetle_UAV.xacro (robot description, xacro)
@@ -1,3 +1,9 @@
 <?xml version="1.0"?>
+<!--
+  Author: Jiaqing "Lance" Wang <jiaqing.wang@sjtu.edu.cn>
+  Shanghai Jiao Tong University, The Nezha Lab
+  Key Laboratory of Polar Ecosystem and Climate Change
+  State Key Laboratory of Submarine Geoscience
+-->
 <robot name="iris" xmlns:xacro="http://ros.org/wiki/xacro">
   <!-- Properties -->

File: src/nezha_sim/nezha_description/nezha_beetle/UUV/nezha_beetle_UUV.xacro (robot description, xacro)
@@ -1,3 +1,9 @@
 <?xml version="1.0"?>
+<!--
+  Author: Jiaqing "Lance" Wang <jiaqing.wang@sjtu.edu.cn>
+  Shanghai Jiao Tong University, The Nezha Lab
+  Key Laboratory of Polar Ecosystem and Climate Change
+  State Key Laboratory of Submarine Geoscience
+-->
 <robot name="nezha_rocket" xmlns:xacro="http://www.ros.org/wiki/xacro" >
 <!-- 1. 定义 / 传入参数 -->

File: src/nezha_sim/nezha_description/nezha_beetle/nezha_beetle_base.xacro (robot description, xacro)
@@ -1,2 +1,8 @@
+<!--
+  Author: Jiaqing "Lance" Wang <jiaqing.wang@sjtu.edu.cn>
+  Shanghai Jiao Tong University, The Nezha Lab
+  Key Laboratory of Polar Ecosystem and Climate Change
+  State Key Laboratory of Submarine Geoscience
+-->
 <robot name="iris" xmlns:xacro="http://ros.org/wiki/xacro">
   <xacro:include filename="$(find nezha_description)/$(arg namespace)/UAV/$(arg namespace)_UAV.xacro" />

File: src/nezha_sim/nezha_description/nezha_beetle/nezha_beetle_plugins.xacro (robot description, xacro)
@@ -1,3 +1,9 @@
 <?xml version="1.0"?>
+<!--
+  Author: Jiaqing "Lance" Wang <jiaqing.wang@sjtu.edu.cn>
+  Shanghai Jiao Tong University, The Nezha Lab
+  Key Laboratory of Polar Ecosystem and Climate Change
+  State Key Laboratory of Submarine Geoscience
+-->
 <robot name="nezha_bettle" xmlns:xacro="http://ros.org/wiki/xacro">
   <xacro:controller_plugin_macro namespace="${namespace}" imu_sub_topic="imu" />

File: src/nezha_sim/nezha_description/nezha_f/UUV/UUV.xacro (robot description, xacro)
@@ -1,3 +1,9 @@
 <?xml version="1.0"?>
+<!--
+  Author: Jiaqing "Lance" Wang <jiaqing.wang@sjtu.edu.cn>
+  Shanghai Jiao Tong University, The Nezha Lab
+  Key Laboratory of Polar Ecosystem and Climate Change
+  State Key Laboratory of Submarine Geoscience
+-->
 <robot xmlns:xacro="http://www.ros.org/wiki/xacro">
   <!--

File: src/nezha_sim/nezha_description/nezha_f/nezha_f_base.xacro (robot description, xacro)
@@ -1,3 +1,9 @@
 <?xml version="1.0"?>
+<!--
+  Author: Jiaqing "Lance" Wang <jiaqing.wang@sjtu.edu.cn>
+  Shanghai Jiao Tong University, The Nezha Lab
+  Key Laboratory of Polar Ecosystem and Climate Change
+  State Key Laboratory of Submarine Geoscience
+-->
 <robot name="nezha_f" xmlns:xacro="http://ros.org/wiki/xacro">
 <xacro:property name="namespace" value="$(arg namespace)" />

File: src/nezha_sim/nezha_description/nezha_f/plugins.xacro (robot description, xacro)
@@ -1,3 +1,9 @@
 <?xml version="1.0"?>
+<!--
+  Author: Jiaqing "Lance" Wang <jiaqing.wang@sjtu.edu.cn>
+  Shanghai Jiao Tong University, The Nezha Lab
+  Key Laboratory of Polar Ecosystem and Climate Change
+  State Key Laboratory of Submarine Geoscience
+-->
 <robot name="plugin" xmlns:xacro="http://www.ros.org/wiki/xacro">
   <xacro:arg name="debug" default="false"/>

File: src/nezha_sim/nezha_description/nezha_gantry_distance/config/materials.xacro (robot description, xacro)
@@ -1,3 +1,9 @@
 <?xml version="1.0"?>
+<!--
+  Author: Jiaqing "Lance" Wang <jiaqing.wang@sjtu.edu.cn>
+  Shanghai Jiao Tong University, The Nezha Lab
+  Key Laboratory of Polar Ecosystem and Climate Change
+  State Key Laboratory of Submarine Geoscience
+-->
 <robot xmlns:xacro="http://www.ros.org/wiki/xacro">
   <material name="blue">

File: src/nezha_sim/nezha_description/nezha_gantry_distance/nezha_gantry.xacro (robot description, xacro)
@@ -1,3 +1,9 @@
 <?xml version="1.0"?>
+<!--
+  Author: Jiaqing "Lance" Wang <jiaqing.wang@sjtu.edu.cn>
+  Shanghai Jiao Tong University, The Nezha Lab
+  Key Laboratory of Polar Ecosystem and Climate Change
+  State Key Laboratory of Submarine Geoscience
+-->
 <robot xmlns:xacro="http://www.ros.org/wiki/xacro" name="gantry_robot">
     <xacro:include filename="$(find nezha_description)/nezha_gantry_velocity/config/materials.xacro" />

File: src/nezha_sim/nezha_description/nezha_gantry_velocity/nezha_gantry.xacro (robot description, xacro)
@@ -1,3 +1,9 @@
 <?xml version="1.0"?>
+<!--
+  Author: Jiaqing "Lance" Wang <jiaqing.wang@sjtu.edu.cn>
+  Shanghai Jiao Tong University, The Nezha Lab
+  Key Laboratory of Polar Ecosystem and Climate Change
+  State Key Laboratory of Submarine Geoscience
+-->
 <robot xmlns:xacro="http://www.ros.org/wiki/xacro" name="nezha_gantry">
   <xacro:include filename="$(find nezha_description)/nezha_gantry_velocity/config/materials.xacro" />

File: src/nezha_sim/nezha_description/nezha_husky/UAV/UAV.xacro (robot description, xacro)
@@ -1,16 +1,28 @@
 <?xml version="1.0"?>
+<!--
+  Author: Jiaqing "Lance" Wang <jiaqing.wang@sjtu.edu.cn>
+  Shanghai Jiao Tong University, The Nezha Lab
+  Key Laboratory of Polar Ecosystem and Climate Change
+  State Key Laboratory of Submarine Geoscience
+-->
 <robot name="iris" xmlns:xacro="http://ros.org/wiki/xacro">
   <!-- Included URDF Files -->
-  <xacro:include filename="$(find nezha_description)/${namespace}/UAV/component_snippets.xacro" />
-  <xacro:include filename="$(find nezha_description)/${namespace}/UAV/UAV_plugin.xacro" />
+  <xacro:include filename="$(find nezha_description)/common/UAV/component_snippets.xacro" />
+  <xacro:include filename="$(find nezha_description)/common/UAV/UAV_plugin.xacro" />
+  <xacro:include filename="$(find nezha_description)/common/UAV/hitl_snippets.xacro" />
   <!-- 从 base.xacro 获取车体尺寸 -->
   <xacro:property name="base_z_size" value="0.24750000" />
   <xacro:property name="horizontal_arm_height" value="0.22" />  <!-- 10cm -->
-  <!-- 原有配置... -->
-  <xacro:controller_plugin_macro namespace="${namespace}" imu_sub_topic="imu" />
+  <!-- Non-HITL: RotorS controller + IMU. Disabled in HITL (real PX4 controls
+       and supplies sensors) to avoid topic/type clashes. -->
+  <xacro:unless value="$(arg enable_mavlink_interface)">
+    <xacro:controller_plugin_macro namespace="${namespace}" imu_sub_topic="imu" />
+    <xacro:default_imu namespace="${namespace}" parent_link="${namespace}/base_link" />
+  </xacro:unless>
+  <!-- HITL: PX4 sensor suite + GPS + mavlink_interface (UAV/flight mode of the
+       transmedia husky). For UGV (rover) HITL use PX4 rover firmware instead. -->
   <xacro:if value="$(arg enable_mavlink_interface)">
-    <xacro:default_mavlink_interface namespace="${namespace}" imu_sub_topic="imu" rotor_count="4" />
+    <xacro:px4_hitl namespace="${namespace}" rotor_count="4" />
   </xacro:if>
-  <xacro:default_imu namespace="${namespace}" parent_link="${namespace}/base_link" />
   <xacro:if value="$(arg enable_ground_truth)">
     <xacro:ground_truth_imu_and_odometry namespace="${namespace}" parent_link="${namespace}/base_link" />

File: src/nezha_sim/nezha_description/nezha_husky/nezha_husky_base.xacro (robot description, xacro)
@@ -1,3 +1,9 @@
 <?xml version="1.0"?>
+<!--
+  Author: Jiaqing "Lance" Wang <jiaqing.wang@sjtu.edu.cn>
+  Shanghai Jiao Tong University, The Nezha Lab
+  Key Laboratory of Polar Ecosystem and Climate Change
+  State Key Laboratory of Submarine Geoscience
+-->
 <robot name="nezha_husky" xmlns:xacro="http://ros.org/wiki/xacro">
   <!-- IMU Link -->

File: src/nezha_sim/nezha_description/nezha_husky1/UAV/UAV.xacro (robot description, xacro)
@@ -1,7 +1,13 @@
 <?xml version="1.0"?>
+<!--
+  Author: Jiaqing "Lance" Wang <jiaqing.wang@sjtu.edu.cn>
+  Shanghai Jiao Tong University, The Nezha Lab
+  Key Laboratory of Polar Ecosystem and Climate Change
+  State Key Laboratory of Submarine Geoscience
+-->
 <robot name="iris" xmlns:xacro="http://ros.org/wiki/xacro">
   <!-- Included URDF Files -->
-  <xacro:include filename="$(find nezha_description)/${namespace}/UAV/component_snippets.xacro" />
-  <xacro:include filename="$(find nezha_description)/${namespace}/UAV/UAV_plugin.xacro" />
+  <xacro:include filename="$(find nezha_description)/common/UAV/component_snippets.xacro" />
+  <xacro:include filename="$(find nezha_description)/common/UAV/UAV_plugin.xacro" />
   <!-- 从 base.xacro 获取车体尺寸 -->
   <xacro:property name="base_z_size" value="0.24750000" />

File: src/nezha_sim/nezha_description/nezha_husky1/UUV/UUV_baselink.xacro (robot description, xacro)
@@ -1,3 +1,9 @@
 <?xml version="1.0"?>
+<!--
+  Author: Jiaqing "Lance" Wang <jiaqing.wang@sjtu.edu.cn>
+  Shanghai Jiao Tong University, The Nezha Lab
+  Key Laboratory of Polar Ecosystem and Climate Change
+  State Key Laboratory of Submarine Geoscience
+-->
 <robot xmlns:xacro="http://www.ros.org/wiki/xacro">
   <!--

File: src/nezha_sim/nezha_description/nezha_husky1/UUV/thruster_snippets.xacro (robot description, xacro)
@@ -1,3 +1,9 @@
 <?xml version="1.0"?>
+<!--
+  Author: Jiaqing "Lance" Wang <jiaqing.wang@sjtu.edu.cn>
+  Shanghai Jiao Tong University, The Nezha Lab
+  Key Laboratory of Polar Ecosystem and Climate Change
+  State Key Laboratory of Submarine Geoscience
+-->
 <robot xmlns:xacro="http://www.ros.org/wiki/xacro">
   <xacro:macro name="box_inertia" params="x y z mass">

File: src/nezha_sim/nezha_description/nezha_husky1/plugins.xacro (robot description, xacro)
@@ -1,2 +1,8 @@
+<!--
+  Author: Jiaqing "Lance" Wang <jiaqing.wang@sjtu.edu.cn>
+  Shanghai Jiao Tong University, The Nezha Lab
+  Key Laboratory of Polar Ecosystem and Climate Change
+  State Key Laboratory of Submarine Geoscience
+-->
 <robot name="plugin" xmlns:xacro="http://www.ros.org/wiki/xacro">
   <xacro:arg name="debug" default="false"/>

File: src/nezha_sim/nezha_description/nezha_mini/UAV/UAV.xacro (robot description, xacro)
@@ -1,15 +1,25 @@
 <?xml version="1.0"?>
+<!--
+  Author: Jiaqing "Lance" Wang <jiaqing.wang@sjtu.edu.cn>
+  Shanghai Jiao Tong University, The Nezha Lab
+  Key Laboratory of Polar Ecosystem and Climate Change
+  State Key Laboratory of Submarine Geoscience
+-->
 <robot name="iris" xmlns:xacro="http://ros.org/wiki/xacro">
   <!-- Included URDF Files -->
-  <xacro:include filename="$(find nezha_description)/${namespace}/UAV/component_snippets.xacro" />
-  <xacro:include filename="$(find nezha_description)/${namespace}/UAV/UAV_plugin.xacro" />
-  <!-- Instantiate a controller. -->
-  <xacro:controller_plugin_macro namespace="${namespace}" imu_sub_topic="imu" />
+  <xacro:include filename="$(find nezha_description)/common/UAV/component_snippets.xacro" />
+  <xacro:include filename="$(find nezha_description)/common/UAV/UAV_plugin.xacro" />
+  <xacro:include filename="$(find nezha_description)/common/UAV/hitl_snippets.xacro" />
+  <!-- Non-HITL: RotorS lee-controller + RotorS IMU. In HITL the real PX4 does
+       control and provides sensors, so these are disabled to avoid clashing on
+       motor-command and /imu topics. -->
+  <xacro:unless value="$(arg enable_mavlink_interface)">
+    <xacro:controller_plugin_macro namespace="${namespace}" imu_sub_topic="imu" />
+    <xacro:default_imu namespace="${namespace}" parent_link="${namespace}/base_link" />
+  </xacro:unless>
+  <!-- HITL: PX4 sensor suite + GPS + mavlink_interface (opens /dev/ttyACM0) -->
   <xacro:if value="$(arg enable_mavlink_interface)">
-    <!-- Instantiate mavlink telemetry interface. -->
-    <xacro:default_mavlink_interface namespace="${namespace}" imu_sub_topic="imu" rotor_count="4" />
+    <xacro:px4_hitl namespace="${namespace}" rotor_count="4" />
   </xacro:if>
-  <!-- Mount an ADIS16448 IMU. -->
-  <xacro:default_imu namespace="${namespace}" parent_link="${namespace}/base_link" />
   <xacro:if value="$(arg enable_ground_truth)">
     <xacro:ground_truth_imu_and_odometry namespace="${namespace}" parent_link="${namespace}/base_link" />

File: src/nezha_sim/nezha_description/nezha_mini/UUV/UUV_baselink.xacro (robot description, xacro)
@@ -1,3 +1,9 @@
 <?xml version="1.0"?>
+<!--
+  Author: Jiaqing "Lance" Wang <jiaqing.wang@sjtu.edu.cn>
+  Shanghai Jiao Tong University, The Nezha Lab
+  Key Laboratory of Polar Ecosystem and Climate Change
+  State Key Laboratory of Submarine Geoscience
+-->
 <robot xmlns:xacro="http://www.ros.org/wiki/xacro">
   <!--

File: src/nezha_sim/nezha_description/nezha_mini/nezha_mini_base.xacro (robot description, xacro)
@@ -1,3 +1,9 @@
 <?xml version="1.0"?>
+<!--
+  Author: Jiaqing "Lance" Wang <jiaqing.wang@sjtu.edu.cn>
+  Shanghai Jiao Tong University, The Nezha Lab
+  Key Laboratory of Polar Ecosystem and Climate Change
+  State Key Laboratory of Submarine Geoscience
+-->
 <robot name="iris" xmlns:xacro="http://ros.org/wiki/xacro">
 <xacro:property name="namespace" value="$(arg namespace)" />
